Commit message: jacobiano init

File: robots_models/puma560_description/urdf/puma560_robot.urdf (robot description, URDF)
Before this commit: robot Puma560, 7 links, 6 joints
Joints:
- joint j1: limit lower=-3.14159265 upper=3.14159265 effort=1000.0 velocity=0 -> lower=-6 upper=6 effort=1000.0 velocity=0
- joint j2: limit lower=-1.570796325 upper=1.570796325 effort=1000.0 velocity=0 -> lower=-6 upper=6 effort=1000.0 velocity=0
- joint j3: limit lower=-1.570796325 upper=1.570796325 effort=1000.0 velocity=0 -> lower=-6 upper=6 effort=1000.0 velocity=0
- joint j4: limit lower=-1.570796325 upper=1.570796325 effort=1000.0 velocity=0 -> lower=-6 upper=6 effort=1000.0 velocity=0
- joint j5: limit lower=-1.570796325 upper=1.570796325 effort=1000.0 velocity=0 -> lower=-6 upper=6 effort=1000.0 velocity=0
- joint j6: limit lower=-1.570796325 upper=1.570796325 effort=1000.0 velocity=0 -> lower=-6 upper=6 effort=1000.0 velocity=0
